File: nuc2f_c.kicad_pcb (KiCad board)
At the start: 4 copper layers, 19.7 x 8.6 mm, 34 parts, among them P1 USB_C_Plug, SW1 SW_Push, U1 STM32F103TBUx, U2 ATECC508A, U3 USBULC6-2M6, U4 NCP114, Y1 8MHz

Commit message: NUC2F-C fix plane fill
Signed-off-by: Dominik Sliwa <dominik@e-plum.pl>
Other:
- board text added: "NUK2F-C v1a"
- board text removed: "NUK2F-C v1"
Changed lines of the file:
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@@
-(kicad_pcb (version 20171130) (host pcbnew 5.0.0-rc2-dev-unknown-r12787-8d017c92)
+(kicad_pcb (version 20171130) (host pcbnew 5.0.0-rc2-dev-unknown-r12853-2eddf1d8)
   (general
     (thickness 0.8)
@@
   (layers
     (0 F.Cu signal)
-    (1 In1.Cu signal hide)
-    (2 In2.Cu signal hide)
+    (1 In1.Cu signal)
+    (2 In2.Cu signal)
     (31 B.Cu signal)
     (32 B.Adhes user)
@@
     (visible_elements FFF9FF1F)
     (pcbplotparams
-      (layerselection 0x00800_7ffffff8)
+      (layerselection 0x01cc0_ffffffff)
       (usegerberextensions false)
       (usegerberattributes false)
@@
     (effects (font (size 0.5 0.5) (thickness 0.1)) (justify mirror))
   )
-  (gr_text "NUK2F-C v1" (at 150.55 76.79 90) (layer Eco1.User)
+  (gr_text "NUK2F-C v1a" (at 150.55 76.79 90) (layer Eco1.User)
     (effects (font (size 0.5 0.5) (thickness 0.1)))
   )

Commit message: NUC2F-C v2
-fix rgb led common voltage
-missing gnd connection on C9
-usb D+ pull-up resistor

Signed-off-by: Dominik Sliwa <dominik@e-plum.pl>
Parts:
- added R5: 1k5, Resistor_SMD:R_0402_1005Metric, F.Cu at (136.2, 78.3)
- moved R6 0.58 mm to (135.3, 79.2), turned to 0 degrees
Connections:
- D1 pad 1: GND -> +3V3
Routing:
- net +3V3: track 17.3 -> 27.6 mm, vias 7 -> 8
- net GND: track 47.1 -> 48.9 mm, vias 16 -> 15
- net Net-(P1-PadA6): track 1.79 -> 3.50 mm
Other:
- board text added: "NUK2F-C v2"
- board text removed: "NUK2F-C v1a"
