File: nuc2f_c.sch (KiCad schematic (older format))
At the start: 8 parts

Commit message: NUC2F-C complete schematics v1
Signed-off-by: Dominik Sliwa <dominik@e-plum.pl>
Parts:
- removed D?: LED_RCBG, symbol Device:LED_RCBG
- removed SW?: SW_Push, symbol Switch:SW_Push
- added C1, C2: 27p, Capacitor_SMD:C_0402_1005Metric, symbol Device:C
- added C10, C12: 2u2, Capacitor_SMD:C_0805_2012Metric, symbol Device:C
- added C11, C13, C3, C4, C5, C6, C7, C8, C9: 100n, Capacitor_SMD:C_0402_1005Metric, symbol Device:C
- added D1: LED_ARGB, LED_SMD:LED_RGB_1210, symbol Device:LED_ARGB
- added D2: LED, LED_SMD:LED_0402_1005Metric, symbol Device:LED
- added R1: 10k, Resistor_SMD:R_0402_1005Metric, symbol Device:R
- added R2, R3, R4, R5: 1k, Resistor_SMD:R_0402_1005Metric, symbol Device:R
- added R6: 5k1, Resistor_SMD:R_0402_1005Metric, symbol Device:R
- added R7, R8: 22R, Resistor_SMD:R_0402_1005Metric, symbol Device:R
- added R9: DNI, Resistor_SMD:R_0402_1005Metric, symbol Device:R
- added SW1: SW_Push, Button_Switch_SMD:SW_SPST_EVQP0, symbol Switch:SW_Push
- added TP1: RST, TestPoint:TestPoint_Pad_D1.0mm, symbol Connector_Specialized:Test_Point
- added TP2: 3.3V, TestPoint:TestPoint_Pad_D1.0mm, symbol Connector_Specialized:Test_Point
- added TP3: GND, TestPoint:TestPoint_Pad_D1.0mm, symbol Connector_Specialized:Test_Point
- added TP4: TX, TestPoint:TestPoint_Pad_D1.0mm, symbol Connector_Specialized:Test_Point
- added TP5: RX, TestPoint:TestPoint_Pad_D1.0mm, symbol Connector_Specialized:Test_Point
- added TP6: SWDIO, TestPoint:TestPoint_Pad_D1.0mm, symbol Connector_Specialized:Test_Point
- added TP7: SWCLK, TestPoint:TestPoint_Pad_D1.0mm, symbol Connector_Specialized:Test_Point
- U1: renamed from U?; footprint VFQFPN36 -> Package_DFN_QFN:QFN-36-1EP_6x6mm_P0.5mm
- U2: renamed from U?; value 24LC00 -> ATECC508A; footprint Package_SOIC:SOIC-8_3.9x4.9mm_P1.27mm -> Package_DFN_QFN:DFN-8-1EP_3x2mm_P0.5mm
- U3: renamed from U?; footprint (none) -> Package_SON:Fairchild_MicroPak-6_1.0x1.45mm_P0.5mm
- U4: renamed from U?; footprint (none) -> Package_DFN_QFN:UDFN-4_1x1mm_P0.65mm
- Y1: renamed from Y?; value Crystal_GND24_Small -> 8MHz; footprint (none) -> Crystal:Crystal_SMD_2016-4Pin_2.0x1.6mm
- gave numbers to parts that had none: 1
Connections:
- net labels added: +3.3V, +5V, D+, D-, GND, I2C_SCL, I2C_SDA
- wire segments 0 -> 171
- no-connect marks 4 -> 25
Other:
- moved on the sheet: U1, U2

Commit message: NUK2F-C assign footprints
Signed-off-by: Dominik Sliwa <dominik@e-plum.pl>
Parts:
- P1: footprint (none) -> Connector_USB:USB_C_Plug_JAE_DX07P024AJ1
- U1: footprint Package_DFN_QFN:QFN-36-1EP_6x6mm_P0.5mm -> Package_DFN_QFN:QFN-36-1EP_6x6mm_P0.5mm_EP3.7x3.7mm
- U2: footprint Package_DFN_QFN:DFN-8-1EP_3x2mm_P0.5mm -> Package_DFN_QFN:DFN-8-1EP_3x2mm_P0.5mm_EP1.36x1.46mm
Changed lines of the file:
@@
 F 0 "P1" H 9820 3348 50  0000 R CNN
 F 1 "USB_C_Plug" H 9820 3439 50  0000 R CNN
-F 2 "" H 10400 3500 50  0001 C CNN
+F 2 "Connector_USB:USB_C_Plug_JAE_DX07P024AJ1" H 10400 3500 50  0001 C CNN
 F 3 "http://www.usb.org/developers/docs/usb_31_033017.zip" H 10400 3500 50  0001 C CNN
 	1    10250 3500
@@
 F 0 "U1" H 2150 3350 50  0000 C CNN
 F 1 "STM32F103TBUx" H 6600 3350 50  0000 C CNN
-F 2 "Package_DFN_QFN:QFN-36-1EP_6x6mm_P0.5mm" H 6900 3275 50  0001 R TNN
+F 2 "Package_DFN_QFN:QFN-36-1EP_6x6mm_P0.5mm_EP3.7x3.7mm" H 6900 3275 50  0001 R TNN
 F 3 "http://www.st.com/st-web-ui/static/active/en/resource/technical/document/datasheet/CD00161566.pdf" H 4500 2200 50  0001 C CNN
 	1    4500 2200
@@
 F 0 "U2" H 5800 7478 50  0000 C CNN
 F 1 "ATECC508A" H 5800 7387 50  0000 C CNN
-F 2 "Package_DFN_QFN:DFN-8-1EP_3x2mm_P0.5mm" H 5850 6750 50  0001 L CNN
+F 2 "Package_DFN_QFN:DFN-8-1EP_3x2mm_P0.5mm_EP1.36x1.46mm" H 5850 6750 50  0001 L CNN
 F 3 "http://ww1.microchip.com/downloads/en/DeviceDoc/21178G.pdf" H 5800 6900 50  0001 C CNN
 	1    5800 7000

Commit message: NUK2F-C schematics v2
Remove power led and few capacitors.

Signed-off-by: Dominik Sliwa <dominik@e-plum.pl>
Parts:
- removed C11: 100n, Capacitor_SMD:C_0402_1005Metric, symbol Device:C
- removed D2: LED, LED_SMD:LED_0402_1005Metric, symbol Device:LED
- removed R5: 1k, Resistor_SMD:R_0402_1005Metric, symbol Device:R
- removed R9: DNI, Resistor_SMD:R_0402_1005Metric, symbol Device:R
- TP1, TP2, TP3, TP4, TP5, TP6, TP7: footprint TestPoint:TestPoint_Pad_D1.0mm -> TestPoint:TestPoint_Pad_D0.5mm
Connections:
- wire segments 171 -> 158
- no-connect marks 25 -> 26
Changed lines of the file:
@@
-$EndComp
-$Comp
-L Device:R R9
-U 1 1 5ADE2D7F
-P 9400 4200
-F 0 "R9" V 9300 4200 50  0000 C CNN
-F 1 "DNI" V 9400 4200 50  0000 C CNN
-F 2 "Resistor_SMD:R_0402_1005Metric" V 9330 4200 50  0001 C CNN
-F 3 "" H 9400 4200 50  0001 C CNN
-	1    9400 4200
-	0    1    1    0
 $EndComp
 $Comp
@@
 L power:GND #PWR0101
 U 1 1 5ADE2E82
-P 8850 4250
-F 0 "#PWR0101" H 8850 4000 50  0001 C CNN
-F 1 "GND" V 8855 4122 50  0000 R CNN
-F 2 "" H 8850 4250 50  0001 C CNN
-F 3 "" H 8850 4250 50  0001 C CNN
-	1    8850 4250
-	0    1    1    0
-$EndComp
-Wire Wire Line
-	9250 4200 9000 4200
-Wire Wire Line
-	9000 4200 9000 4250
-Wire Wire Line
-	9000 4300 9050 4300
-Wire Wire Line
-	8850 4250 9000 4250
-Connection ~ 9000 4250
-Wire Wire Line
-	9000 4250 9000 4300
-Wire Wire Line
-	9550 4200 9650 4200
+P 8850 4300
+F 0 "#PWR0101" H 8850 4050 50  0001 C CNN
+F 1 "GND" V 8855 4172 50  0000 R CNN
+F 2 "" H 8850 4300 50  0001 C CNN
+F 3 "" H 8850 4300 50  0001 C CNN
+	1    8850 4300
+	0    1    1    0
+$EndComp
 Wire Wire Line
 	9650 4300 9350 4300
@@
 	1    0    0    -1
 $EndComp
-$Comp
-L Device:C C11
-U 1 1 5ADE78F3
-P 10350 5750
-F 0 "C11" H 10465 5796 50  0000 L CNN
-F 1 "100n" H 10465 5705 50  0000 L CNN
-F 2 "Capacitor_SMD:C_0402_1005Metric" H 10388 5600 50  0001 C CNN
-F 3 "" H 10350 5750 50  0001 C CNN
-	1    10350 5750
-	1    0    0    -1
-$EndComp
 Wire Wire Line
 	10750 5600 10750 5550
-Wire Wire Line
-	10750 5550 10350 5550
-Wire Wire Line
-	10350 5600 10350 5550
-Connection ~ 10350 5550
-Wire Wire Line
-	10350 5550 10100 5550
 $Comp
 L power:+5V #PWR0105
@@
 Wire Wire Line
 	10750 5950 10750 5900
-Wire Wire Line
-	10750 5950 10350 5950
 $Comp
 L Device:C C5
@@
 	9950 5950 9550 5950
 Wire Wire Line
-	10350 5900 10350 5950
-Connection ~ 10350 5950
-Wire Wire Line
-	10350 5950 9950 5950
-Wire Wire Line
 	9150 5550 9050 5550
 Wire Wire Line
@@
 Wire Wire Line
 	9050 5550 8850 5550
-$Comp
-L Device:LED D2
-U 1 1 5AE00DEC
-P 6750 5700
-F 0 "D2" V 6788 5583 50  0000 R CNN
-F 1 "LED" V 6697 5583 50  0000 R CNN
-F 2 "LED_SMD:LED_0402_1005Metric" H 6750 5700 50  0001 C CNN
-F 3 "~" H 6750 5700 50  0001 C CNN
-	1    6750 5700
-	0    -1   -1   0
-$EndComp
-$Comp
-L Device:R R5
-U 1 1 5AE01071
-P 7050 5550
-F 0 "R5" V 6950 5550 50  0000 C CNN
-F 1 "1k" V 7050 5550 50  0000 C CNN
-F 2 "Resistor_SMD:R_0402_1005Metric" V 6980 5550 50  0001 C CNN
-F 3 "" H 7050 5550 50  0001 C CNN
-	1    7050 5550
-	0    1    1    0
-$EndComp
-Wire Wire Line
-	7300 5550 7200 5550
-Connection ~ 7300 5550
-Wire Wire Line
-	7300 5950 6750 5950
-Wire Wire Line
-	6750 5950 6750 5850
-Connection ~ 7300 5950
-Wire Wire Line
-	6900 5550 6750 5550
 Wire Wire Line
 	6200 6900 6600 6900
@@
 F 0 "TP6" V 7250 2875 50  0000 L CNN
 F 1 "SWDIO" V 7325 2900 50  0000 L CNN
-F 2 "TestPoint:TestPoint_Pad_D1.0mm" H 7525 2700 50  0001 C CNN
+F 2 "TestPoint:TestPoint_Pad_D0.5mm" H 7525 2700 50  0001 C CNN
 F 3 "~" H 7525 2700 50  0001 C CNN
 	1    7325 2700
@@
 F 0 "TP7" V 7400 2975 50  0000 L CNN
 F 1 "SWCLK" V 7325 3000 50  0000 L CNN
-F 2 "TestPoint:TestPoint_Pad_D1.0mm" H 7525 2800 50  0001 C CNN
+F 2 "TestPoint:TestPoint_Pad_D0.5mm" H 7525 2800 50  0001 C CNN
 F 3 "~" H 7525 2800 50  0001 C CNN
 	1    7325 2800
@@
 F 0 "TP1" V 1800 1575 50  0000 L CNN
 F 1 "RST" V 1875 1600 50  0000 L CNN
-F 2 "TestPoint:TestPoint_Pad_D1.0mm" H 2075 1400 50  0001 C CNN
+F 2 "TestPoint:TestPoint_Pad_D0.5mm" H 2075 1400 50  0001 C CNN
 F 3 "~" H 2075 1400 50  0001 C CNN
 	1    1875 1400
@@
 F 0 "TP2" V 4650 1075 50  0000 L CNN
 F 1 "3.3V" V 4725 1100 50  0000 L CNN
-F 2 "TestPoint:TestPoint_Pad_D1.0mm" H 4925 900 50  0001 C CNN
+F 2 "TestPoint:TestPoint_Pad_D0.5mm" H 4925 900 50  0001 C CNN
 F 3 "~" H 4925 900 50  0001 C CNN
 	1    4725 900
@@
 F 0 "TP3" V 4750 3575 50  0000 L CNN
 F 1 "GND" V 4825 3600 50  0000 L CNN
-F 2 "TestPoint:TestPoint_Pad_D1.0mm" H 5025 3400 50  0001 C CNN
+F 2 "TestPoint:TestPoint_Pad_D0.5mm" H 5025 3400 50  0001 C CNN
 F 3 "~" H 5025 3400 50  0001 C CNN
 	1    4825 3400
@@
 F 0 "TP4" V 7250 2475 50  0000 L CNN
 F 1 "TX" V 7325 2500 50  0000 L CNN
-F 2 "TestPoint:TestPoint_Pad_D1.0mm" H 7525 2300 50  0001 C CNN
+F 2 "TestPoint:TestPoint_Pad_D0.5mm" H 7525 2300 50  0001 C CNN
 F 3 "~" H 7525 2300 50  0001 C CNN
 	1    7325 2300
@@
 F 0 "TP5" V 7400 2575 50  0000 L CNN
 F 1 "RX" V 7325 2600 50  0000 L CNN
-F 2 "TestPoint:TestPoint_Pad_D1.0mm" H 7525 2400 50  0001 C CNN
+F 2 "TestPoint:TestPoint_Pad_D0.5mm" H 7525 2400 50  0001 C CNN
 F 3 "~" H 7525 2400 50  0001 C CNN
 	1    7325 2400
@@
 Wire Wire Line
 	7525 3900 7650 3900
+Wire Wire Line
+	10100 5550 10750 5550
+Wire Wire Line
+	9950 5950 10750 5950
+NoConn ~ 9650 4200
+Wire Wire Line
+	8850 4300 9050 4300
 $EndSCHEMATC

Commit message: NUC2F-C v2
-fix rgb led common voltage
-missing gnd connection on C9
-usb D+ pull-up resistor

Signed-off-by: Dominik Sliwa <dominik@e-plum.pl>
Parts:
- added R5: 1k5, Resistor_SMD:R_0402_1005Metric, symbol Device:R
Connections:
- wire segments 158 -> 162
Changed lines of the file:
@@
 	10250 1800 10150 1800
 Wire Wire Line
-	9500 3800 9650 3800
+	9500 3800 9550 3800
 Wire Wire Line
 	9650 4000 9500 4000
@@
 Wire Wire Line
 	875  2775 775  2775
-$Comp
-L power:GND #PWR0118
-U 1 1 5AEFB8FB
-P 1550 3950
-F 0 "#PWR0118" H 1550 3700 50  0001 C CNN
-F 1 "GND" H 1555 3777 50  0000 C CNN
-F 2 "" H 1550 3950 50  0001 C CNN
-F 3 "" H 1550 3950 50  0001 C CNN
-	1    1550 3950
-	1    0    0    -1
-$EndComp
 $Comp
 L Device:R R2
@@
 Wire Wire Line
 	8850 4300 9050 4300
+$Comp
+L power:+3.3V #PWR0118
+U 1 1 5AEFDB80
+P 1550 3950
+F 0 "#PWR0118" H 1550 3800 50  0001 C CNN
+F 1 "+3.3V" H 1565 4123 50  0000 C CNN
+F 2 "" H 1550 3950 50  0001 C CNN
+F 3 "" H 1550 3950 50  0001 C CNN
+	1    1550 3950
+	-1   0    0    1
+$EndComp
+$Comp
+L Device:R R5
+U 1 1 5AF52896
+P 9350 3600
+F 0 "R5" V 9250 3600 50  0000 C CNN
+F 1 "1k5" V 9350 3600 50  0000 C CNN
+F 2 "Resistor_SMD:R_0402_1005Metric" V 9280 3600 50  0001 C CNN
+F 3 "" H 9350 3600 50  0001 C CNN
+	1    9350 3600
+	0    1    1    0
+$EndComp
+Wire Wire Line
+	9500 3600 9550 3600
+Wire Wire Line
+	9550 3600 9550 3800
+Connection ~ 9550 3800
+Wire Wire Line
+	9550 3800 9650 3800
+$Comp
+L power:+3.3V #PWR0120
+U 1 1 5AF5B0D5
+P 9100 3600
+F 0 "#PWR0120" H 9100 3450 50  0001 C CNN
+F 1 "+3.3V" H 9115 3773 50  0000 C CNN
+F 2 "" H 9100 3600 50  0001 C CNN
+F 3 "" H 9100 3600 50  0001 C CNN
+	1    9100 3600
+	0    -1   -1   0
+$EndComp
+Wire Wire Line
+	9100 3600 9200 3600
 $EndSCHEMATC
